Commit message: feat: add camera to go2

File: go2_description/xacro/gazebo.xacro (robot description, xacro)
@@ -58,4 +58,60 @@
             <pose>0 0 0 0 0 0</pose>
         </sensor>
+    </gazebo>
+    <!-- Camera -->
+    <!-- 相機 Joint -->
+    <joint name="camera_joint" type="fixed">
+        <parent link="trunk"/>
+        <child link="camera_link"/>
+        <origin xyz="0.32 0.0 0.085" rpy="0 0.35 0"/> <!--相機角度向下20deg-->
+    </joint>
+    <!-- 相機 Link -->
+    <link name="camera_link">
+        <inertial>
+            <mass value="0.001"/>
+            <origin xyz="0 0 0" rpy="0 0 0"/>
+            <inertia ixx="1e-6" iyy="1e-6" izz="1e-6" ixy="0" ixz="0" iyz="0"/>
+        </inertial>
+        <visual>
+            <origin xyz="0 0 0" rpy="0 0 0"/>
+            <geometry>
+                <box size="0.025 0.09 0.025"/>
+            </geometry>
+            <material name="green"/>
+        </visual>
+    </link>
+    <!-- 相機 Setting -->
+    <gazebo reference="camera_link">
+    <sensor name="depth_camera" type="depth">
+        <always_on>true</always_on>
+        <update_rate>30</update_rate>
+        <visualize>true</visualize>
+        <pose>0 0 0 0 0 0</pose>
+        <camera>
+            <horizontal_fov>1.5</horizontal_fov> <!--86 deg-->
+            <image>
+                <width>640</width>
+                <height>480</height>
+                <format>R8G8B8</format>
+            </image>
+            <depth_image>
+                <width>640</width>
+                <height>480</height>
+                <format>FLOAT32</format>
+            </depth_image>
+            <clip>
+                <near>0.1</near>
+                <far>10</far>
+            </clip>
+        </camera>
+        <plugin name="depth_camera_controller" filename="libgazebo_ros_depth_camera.so">
+            <robotNamespace>/go2</robotNamespace>
+            <cameraName>depth_cam</cameraName>
+            <imageTopicName>/camera/image_raw</imageTopicName>
+            <depthImageTopicName>/camera/forward_depth</depthImageTopicName>
+            <cameraInfoTopicName>/camera/camera_info</cameraInfoTopicName>
+            <frameName>camera_link</frameName>
+        </plugin>
+    </sensor>
     </gazebo>
     <!-- Foot contacts. -->
